File: inyector-audio/diseños-kicad/inyector-audio/inyector-audio.sch (KiCad schematic (older format))
At the start: 11 parts, among them J1 Ent, J2 Sal, U1 NE555

Commit message: Add files via upload
Parts:
- removed TS1: t1, Mis_Simbolos:Taladro_sujecion_3mm, symbol Mis_Simbolos:Taladro_sujeccion_3mm
- removed TS2, TS3, TS4: Taladro_sujeccion_3mm, Mis_Simbolos:Taladro_sujecion_3mm, symbol Mis_Simbolos:Taladro_sujeccion_3mm
Other:
- note removed: "Agujeros de sujecion"
Changed lines of the file:
@@
 Sheet 1 1
 Title "Inyector de audio"
-Date "2021-06-15"
-Rev "1.0"
+Date "2021-06-18"
+Rev "2.0"
 Comp "Electronica reciclada"
 Comment1 ""
@@
 Wire Wire Line
 	5250 2600 5650 2600
-$Comp
-L Mis_Simbolos:Taladro_sujeccion_3mm TS1
-U 1 1 60C9AB22
-P 8600 3300
-F 0 "TS1" H 8550 3450 50  0000 L CNN
-F 1 "t1" H 8699 3208 50  0001 L CNN
-F 2 "Mis_Simbolos:Taladro_sujecion_3mm" H 8600 3300 50  0001 C CNN
-F 3 "" H 8600 3300 50  0001 C CNN
-	1    8600 3300
-	1    0    0    -1
-$EndComp
-$Comp
-L Mis_Simbolos:Taladro_sujeccion_3mm TS2
-U 1 1 60C9AF25
-P 9000 3300
-F 0 "TS2" H 8950 3450 50  0000 L CNN
-F 1 "Taladro_sujeccion_3mm" H 9099 3208 50  0001 L CNN
-F 2 "Mis_Simbolos:Taladro_sujecion_3mm" H 9000 3300 50  0001 C CNN
-F 3 "" H 9000 3300 50  0001 C CNN
-	1    9000 3300
-	1    0    0    -1
-$EndComp
-$Comp
-L Mis_Simbolos:Taladro_sujeccion_3mm TS3
-U 1 1 60C9B7B0
-P 9450 3300
-F 0 "TS3" H 9400 3450 50  0000 L CNN
-F 1 "Taladro_sujeccion_3mm" H 9549 3208 50  0001 L CNN
-F 2 "Mis_Simbolos:Taladro_sujecion_3mm" H 9450 3300 50  0001 C CNN
-F 3 "" H 9450 3300 50  0001 C CNN
-	1    9450 3300
-	1    0    0    -1
-$EndComp
-$Comp
-L Mis_Simbolos:Taladro_sujeccion_3mm TS4
-U 1 1 60C9BE1E
-P 9900 3300
-F 0 "TS4" H 9850 3450 50  0000 L CNN
-F 1 "Taladro_sujeccion_3mm" H 9999 3208 50  0001 L CNN
-F 2 "Mis_Simbolos:Taladro_sujecion_3mm" H 9900 3300 50  0001 C CNN
-F 3 "" H 9900 3300 50  0001 C CNN
-	1    9900 3300
-	1    0    0    -1
-$EndComp
-Wire Notes Line
-	8250 2850 10350 2850
-Wire Notes Line
-	10350 2850 10350 3600
-Wire Notes Line
-	10350 3600 8250 3600
-Wire Notes Line
-	8250 3600 8250 2850
-Text Notes 8400 3000 0    50   ~ 0
-Agujeros de sujecion
 $EndSCHEMATC

Commit message: Add files via upload
Parts:
- added SW1: SW_DIP_x01, Connector_PinHeader_2.00mm:PinHeader_1x02_P2.00mm_Vertical, symbol Switch:SW_DIP_x01
- J1, J2: footprint TerminalBlock:TerminalBlock_Altech_AK300-2_P5.00mm -> Connector_PinHeader_2.00mm:PinHeader_1x02_P2.00mm_Vertical
Connections:
- net +9V: now also SW1.2; no longer J1.2 (Pin_2)
- new net: J1.2 (Pin_2), SW1.1
Other:
- moved on the sheet: J1
Changed lines of the file:
@@
 Sheet 1 1
 Title "Inyector de audio"
-Date "2021-06-18"
-Rev "2.0"
+Date "2021-06-23"
+Rev "4.0"
 Comp "Electronica reciclada"
 Comment1 ""
@@
 F 0 "J2" H 6830 3492 50  0000 L CNN
 F 1 "Sal" H 6830 3401 50  0000 L CNN
-F 2 "TerminalBlock:TerminalBlock_Altech_AK300-2_P5.00mm" H 6750 3500 50  0001 C CNN
+F 2 "Connector_PinHeader_2.00mm:PinHeader_1x02_P2.00mm_Vertical" H 6750 3500 50  0001 C CNN
 F 3 "~" H 6750 3500 50  0001 C CNN
 	1    6750 3500
@@
 L Connector:Screw_Terminal_01x02 J1
 U 1 1 5F3C7084
-P 2250 3700
-F 0 "J1" H 2170 3375 50  0000 C CNN
-F 1 "Ent" H 2170 3466 50  0000 C CNN
-F 2 "TerminalBlock:TerminalBlock_Altech_AK300-2_P5.00mm" H 2250 3700 50  0001 C CNN
-F 3 "~" H 2250 3700 50  0001 C CNN
-	1    2250 3700
+P 1700 3700
+F 0 "J1" H 1620 3375 50  0000 C CNN
+F 1 "Ent" H 1620 3466 50  0000 C CNN
+F 2 "Connector_PinHeader_2.00mm:PinHeader_1x02_P2.00mm_Vertical" H 1700 3700 50  0001 C CNN
+F 3 "~" H 1700 3700 50  0001 C CNN
+	1    1700 3700
 	-1   0    0    1
 $EndComp
 Wire Wire Line
 	3700 2600 2950 2600
-Wire Wire Line
-	2950 2600 2950 3600
-Wire Wire Line
-	2950 3600 2450 3600
 Connection ~ 3700 2600
-Wire Wire Line
-	2450 3700 2950 3700
 Wire Wire Line
 	2950 3700 2950 4700
@@
 Wire Wire Line
 	5250 2600 5650 2600
+$Comp
+L Switch:SW_DIP_x01 SW1
+U 1 1 60D24622
+P 2400 3500
+F 0 "SW1" H 2400 3767 50  0000 C CNN
+F 1 "SW_DIP_x01" H 2400 3676 50  0000 C CNN
+F 2 "Connector_PinHeader_2.00mm:PinHeader_1x02_P2.00mm_Vertical" H 2400 3500 50  0001 C CNN
+F 3 "~" H 2400 3500 50  0001 C CNN
+	1    2400 3500
+	1    0    0    -1
+$EndComp
+Wire Wire Line
+	1900 3700 2950 3700
+Wire Wire Line
+	1900 3600 2000 3600
+Wire Wire Line
+	2000 3600 2000 3500
+Wire Wire Line
+	2000 3500 2100 3500
+Wire Wire Line
+	2700 3500 2950 3500
+Wire Wire Line
+	2950 3500 2950 2600
 $EndSCHEMATC
